Commit message: fixes for navigation also, enabling 5 depth cameras uses a lot of computing resources, use gihly reliable velodyne lidar instead

File: resource/rd_spot.urdf (robot description, URDF)
Before this commit: robot Spot, 69 links, 68 joints
Links:
- removed link HokuyoUrg04lxug01
- removed link Kinect
- added link Velodyne_Puck; collision cylinder length=0.0727 radius=0.052; visual cylinder length=0.0727 radius=0.052
Joints:
- removed joint base_link_HokuyoUrg04lxug01_joint
- removed joint base_link_Kinect_joint
- removed joint distance sensor_solid_0_joint
- removed joint solid_kinect color_joint
- removed joint solid_kinect range_joint
- removed joint tilt motor
- added joint base_link_Velodyne_Puck_joint: type fixed, parent base_link, child Velodyne_Puck, origin xyz=-0.063 0 0.1518 rpy=-0.000008 -0.000008 0.000001
- added joint base_link_solid_0_joint: type fixed, parent base_link, child solid_0, origin xyz=0.496831 0.000001 0.104801 rpy=1.2208 -0.00001 -1.570793
- added joint distance sensor_solid_joint: type fixed, parent distance sensor, child solid, origin xyz=0 0 0 rpy=0 0 0
- added joint solid_0_kinect color_joint: type fixed, parent solid_0, child kinect color, origin xyz=0 0 -0.0127 rpy=-0.785397 1.570792 0.785397
- added joint solid_0_kinect range_joint: type fixed, parent solid_0, child kinect range, origin xyz=0 0 -0.0127 rpy=-0.785397 1.570792 0.785397
- joint rear left piston motor: child solid_1 -> solid_2
- joint rear right piston motor: child solid_2 -> solid_1

Commit message: fixes for navigation also, enabling 5 depth cameras uses a lot of computing resources, use gihly reliable velodyne lidar instead

File: resource/rd_spot.urdf (robot description, URDF)
Before this commit: robot Spot, 38 links, 37 joints
Links:
- added link Velodyne_Puck; collision cylinder length=0.0727 radius=0.052; visual cylinder length=0.0727 radius=0.052
- added link distance_sensor
- added link kinect; collision box size=0.084 0.027 0.068; visual box size=0.084 0.027 0.068
- added link kinect color
- added link kinect range
- added link left flank depth
- added link left head depth
- added link rear depth
- added link right flank depth
- added link right head depth
- added link solid_3
- added link solid_4
Joints:
- added joint base_link_Velodyne_Puck_joint: type fixed, parent base_link, child Velodyne_Puck, origin xyz=0.336 0.000001 0.1518 rpy=-0.000008 -0.000008 0.000001
- added joint base_link_kinect_joint: type fixed, parent base_link, child kinect, origin xyz=0.334809 -0.000999 0.180133 rpy=-0.000011 0.008756 0.000004
- added joint base_link_left flank depth_joint: type fixed, parent base_link, child left flank depth, origin xyz=-0.13568 0.110127 0.065528 rpy=-0.000003 0.403191 1.570802
- added joint base_link_left head depth_joint: type fixed, parent base_link, child left head depth, origin xyz=0.46325 0.045111 0.029551 rpy=-0.158862 0.433786 -0.408004
- added joint base_link_rear depth_joint: type fixed, parent base_link, child rear depth, origin xyz=-0.278136 -1.397633 0.628752 rpy=0.000015 0.474984 -3.141579
- added joint base_link_right flank depth_joint: type fixed, parent base_link, child right flank depth, origin xyz=-0.135678 -0.110163 0.06561 rpy=0.000005 0.413171 -1.570794
- added joint base_link_right head depth_joint: type fixed, parent base_link, child right head depth, origin xyz=0.462603 -0.044896 0.027972 rpy=0.193959 0.3931 0.409605
- added joint base_link_solid_joint: type fixed, parent base_link, child solid, origin xyz=0.416 0 0.111801 rpy=-0.000008 -0.000008 0.000001
- added joint solid_0_kinect color_joint: type fixed, parent solid_0, child kinect color, origin xyz=0 0 -0.0127 rpy=-0.785397 1.570792 0.785397
- added joint solid_0_kinect range_joint: type fixed, parent solid_0, child kinect range, origin xyz=0 0 -0.0127 rpy=-0.785397 1.570792 0.785397
- added joint solid_distance_sensor_joint: type fixed, parent solid, child distance_sensor, origin xyz=0 0 0 rpy=0 0.000005 0
- added joint tilt motor: type revolute, parent kinect, child solid_0, origin xyz=0 0 0.05 rpy=1.570741 0.000118 -1.570741, axis 1 0.000118 0.000055, limit lower=-0.47 upper=0.47 effort=10 velocity=10
- joint base_link_rear camera_joint: origin xyz=-0.278136 -1.397633 0.628752 rpy=0.000015 0.474984 -3.141579 -> xyz=-0.448136 -0.018115 0.012558 rpy=0.000015 0.474984 -3.141579
- joint front left piston motor: child solid_2 -> solid_4
- joint front right piston motor: child solid_1 -> solid_3
- joint rear left piston motor: child solid_0 -> solid_2
- joint rear right piston motor: child solid -> solid_1

Commit message: move example scripts to separate folder
also some moveit related fixes

File: resource/rd_spot.urdf (robot description, URDF)
Before this commit: robot Spot, 68 links, 67 joints
Links:
- removed link ROBOTIQ 3f Gripper
- added link Robotiq3fGripper; collision box size=0.126 0.093 0.13; collision cylinder length=0.05 radius=0.023
Joints:
- removed joint wrist_3_link_ROBOTIQ 3f Gripper_joint
- added joint wrist_3_link_Robotiq3fGripper_joint: type fixed, parent wrist_3_link, child Robotiq3fGripper, origin xyz=0 0.13 0 rpy=0 0 0
- joint finger_middle_joint_1: parent ROBOTIQ 3f Gripper -> Robotiq3fGripper
- joint palm_finger_1_joint: parent ROBOTIQ 3f Gripper -> Robotiq3fGripper
- joint palm_finger_2_joint: parent ROBOTIQ 3f Gripper -> Robotiq3fGripper

Commit message: use spot's arm lookalike with tiagogripper

File: resource/rd_spot.urdf (robot description, URDF)
Before this commit: robot Spot, 68 links, 67 joints
Links:
- removed link Robotiq3fGripper
- removed link UR3e
- removed link distance sensor
- removed link finger_1_link_0
- removed link finger_1_link_1
- removed link finger_1_link_2
- removed link finger_1_link_3
- removed link finger_2_link_0
- removed link finger_2_link_1
- removed link finger_2_link_2
- removed link finger_2_link_3
- removed link finger_middle_link_1
- removed link finger_middle_link_2
- removed link finger_middle_link_3
- removed link forearm_link
- removed link shoulder_link
- removed link solid_4
- removed link upper_arm_link
- removed link wrist_1_link
- removed link wrist_2_link
- removed link wrist_3_link
- added link SpotArm; collision cylinder length=0.035 radius=0.075; visual cylinder length=0.035 radius=0.075
- added link cap screw
- added link cap screw(1)
- added link cap screw(10)
- added link cap screw(11)
- added link cap screw(12)
- added link cap screw(13)
- added link cap screw(14)
- added link cap screw(15)
- added link cap screw(16)
- added link cap screw(17)
- added link cap screw(18)
- added link cap screw(19)
- added link cap screw(2)
- added link cap screw(3)
- added link cap screw(4)
- added link cap screw(5)
- added link cap screw(6)
- added link cap screw(7)
- added link cap screw(8)
- added link cap screw(9)
- added link front; collision box size=0.04 0.0217 0.105; collision box size=0.04 0.0217 0.105
- added link gripper_left_finger_link; collision box size=0.0055 0.0295 0.018; collision box size=0.0076 0.05091 0.08982
- added link gripper_right_finger_link; collision box size=0.0055 0.0295 0.018; collision box size=0.0076 0.05091 0.08982
- added link spotarm_link1; collision box size=0.14 0.01 0.08; collision box size=0.14 0.01 0.08
- added link spotarm_link2; collision box size=0.06 0.059 0.093; collision cylinder length=0.24 radius=0.0456
- added link spotarm_link3; collision box size=0.16 0.041 0.04; collision cylinder length=0.059 radius=0.0477
- added link spotarm_link4
- added link spotarm_link5; collision box size=0.04 0.044 0.042; collision cylinder length=0.21 radius=0.0477
- added link spotarm_link6; collision cylinder length=0.065 radius=0.0477; visual cylinder length=0.065 radius=0.0477
Joints:
- removed joint base_link_UR3e_joint
- removed joint base_link_distance sensor_joint
- removed joint base_link_solid_0_joint
- removed joint distance sensor_solid_joint
- removed joint elbow_joint
- removed joint finger_1_joint_1
- removed joint finger_1_joint_2
- removed joint finger_1_joint_3
- removed joint finger_2_joint_1
- removed joint finger_2_joint_2
- removed joint finger_2_joint_3
- removed joint finger_middle_joint_1
- removed joint finger_middle_joint_2
- removed joint finger_middle_joint_3
- removed joint palm_finger_1_joint
- removed joint palm_finger_2_joint
- removed joint shoulder_lift_joint
- removed joint shoulder_pan_joint
- removed joint solid_0_kinect color_joint
- removed joint solid_0_kinect range_joint
- removed joint wrist_1_joint
- removed joint wrist_2_joint
- removed joint wrist_3_joint
- removed joint wrist_3_link_Robotiq3fGripper_joint
- added joint Slider11: type prismatic, parent spotarm_link4, child spotarm_link5, origin xyz=0.035 0 0 rpy=0 0 0, axis 0 0 1, limit lower=0 upper=0.075 effort=100 velocity=100
- added joint base_link_SpotArm_joint: type fixed, parent base_link, child SpotArm, origin xyz=0.35 0 0.1118 rpy=-0.000017 -0.000003 0.000005
- added joint base_link_solid_joint: type fixed, parent base_link, child solid, origin xyz=0.496831 0.000001 0.104801 rpy=1.2208 -0.00001 -1.570793
- added joint front_cap screw(1)_joint: type fixed, parent front, child cap screw(1), origin xyz=0.0477 0.008 -0.043 rpy=3.141593 -1.570793 3.141593
- added joint front_cap screw(10)_joint: type fixed, parent front, child cap screw(10), origin xyz=-0.0477 -0.008 -0.043 rpy=3.141593 1.570793 3.141593
- added joint front_cap screw(11)_joint: type fixed, parent front, child cap screw(11), origin xyz=-0.0477 -0.008 -0.0108 rpy=3.141593 1.570793 3.141593
- added joint front_cap screw(12)_joint: type fixed, parent front, child cap screw(12), origin xyz=-0.0425 0.0094 -0.0945 rpy=0 0 0
- added joint front_cap screw(13)_joint: type fixed, parent front, child cap screw(13), origin xyz=0.0426 -0.0094 -0.09448 rpy=0 0 0
- added joint front_cap screw(14)_joint: type fixed, parent front, child cap screw(14), origin xyz=0 -0.033 0.0026 rpy=3.14159 0 0
- added joint front_cap screw(15)_joint: type fixed, parent front, child cap screw(15), origin xyz=0 0.033 0.0026 rpy=3.14159 0 0
- added joint front_cap screw(16)_joint: type fixed, parent front, child cap screw(16), origin xyz=-0.0433 -0.0315 0.0026 rpy=3.14159 0 0
- added joint front_cap screw(17)_joint: type fixed, parent front, child cap screw(17), origin xyz=0.0433 0.0315 0.0026 rpy=3.14159 0 0
- added joint front_cap screw(18)_joint: type fixed, parent front, child cap screw(18), origin xyz=-0.0415 0.0029 -0.0004 rpy=3.14159 0 0
- added joint front_cap screw(19)_joint: type fixed, parent front, child cap screw(19), origin xyz=0.0415 -0.0029 -0.0004 rpy=3.14159 0 0
- added joint front_cap screw(2)_joint: type fixed, parent front, child cap screw(2), origin xyz=0.0477 0.008 -0.075 rpy=3.141593 -1.570793 3.141593
- added joint front_cap screw(3)_joint: type fixed, parent front, child cap screw(3), origin xyz=0.0477 -0.008 -0.075 rpy=3.141593 -1.570793 3.141593
- added joint front_cap screw(4)_joint: type fixed, parent front, child cap screw(4), origin xyz=0.0477 -0.008 -0.043 rpy=3.141593 -1.570793 3.141593
- added joint front_cap screw(5)_joint: type fixed, parent front, child cap screw(5), origin xyz=0.0477 -0.008 -0.0108 rpy=3.141593 -1.570793 3.141593
- added joint front_cap screw(6)_joint: type fixed, parent front, child cap screw(6), origin xyz=-0.0477 0.008 -0.0108 rpy=3.141593 1.570793 3.141593
- added joint front_cap screw(7)_joint: type fixed, parent front, child cap screw(7), origin xyz=-0.0477 0.008 -0.043 rpy=3.141593 1.570793 3.141593
- added joint front_cap screw(8)_joint: type fixed, parent front, child cap screw(8), origin xyz=-0.0477 0.008 -0.075 rpy=3.141593 1.570793 3.141593
- added joint front_cap screw(9)_joint: type fixed, parent front, child cap screw(9), origin xyz=-0.0477 -0.008 -0.075 rpy=3.141593 1.570793 3.141593
- added joint front_cap screw_joint: type fixed, parent front, child cap screw, origin xyz=0.0477 0.008 -0.0108 rpy=3.141593 -1.570793 3.141593
- added joint gripper_left_finger_joint: type prismatic, parent front, child gripper_left_finger_link, origin xyz=0 0 0 rpy=0 0 3.1415, axis 1 0.000093 0, limit lower=0 upper=0.045 effort=16 velocity=0.05
- added joint gripper_right_finger_joint: type prismatic, parent front, child gripper_right_finger_link, origin xyz=0 0.0005 -0.007 rpy=0 0 0, axis 1 0 0, limit lower=0 upper=0.045 effort=16 velocity=0.05
- added joint solid_kinect color_joint: type fixed, parent solid, child kinect color, origin xyz=0 0 -0.0127 rpy=-2.356193 1.570792 -0.7854
- added joint solid_kinect range_joint: type fixed, parent solid, child kinect range, origin xyz=0 0 -0.0127 rpy=-0.785397 1.570792 0.785397
- added joint spotarm_1_joint: type revolute, parent SpotArm, child spotarm_link1, origin xyz=0 0 0.04 rpy=0 0 0, axis 0 0 1, limit lower=-2.61799 upper=3.14159 effort=500 velocity=0.5
- added joint spotarm_2_joint: type revolute, parent spotarm_link1, child spotarm_link2, origin xyz=0 0.03 0.1 rpy=0 0 0, axis 0 -1 0, limit lower=-0.523599 upper=3.14159 effort=500 velocity=0.5
- added joint spotarm_3_joint: type revolute, parent spotarm_link2, child spotarm_link3, origin xyz=0.3385 -0.02 0.000137 rpy=0 0 0, axis 0 1 0, limit lower=0 upper=2.61799 effort=500 velocity=0.5
- added joint spotarm_4_joint: type revolute, parent spotarm_link3, child spotarm_link4, origin xyz=0.107 -0.01 0.09734 rpy=0 0 0, axis 1 0 0, limit lower=-4.3633 upper=1.22173 effort=500 velocity=0.5
- added joint spotarm_5_joint: type revolute, parent spotarm_link5, child spotarm_link6, origin xyz=0.2413 0.01 0 rpy=0 0 0, axis 0 1 0, limit lower=-1.0472 upper=1.0472 effort=500 velocity=0.5
- added joint spotarm_6_joint: type revolute, parent spotarm_link6, child front, origin xyz=0.1 -0.0105 0 rpy=3.141593 -1.570793 3.141593, axis 0.000004 0 1, limit lower=-4.45059 upper=1.30899 effort=500 velocity=0.5
- joint base_link_left flank camera_joint: origin xyz=-0.13568 0.110127 0.065528 rpy=-0.000003 0.403191 1.570802 -> xyz=-0.13568 0.110127 0.065528 rpy=-1.570799 0.403191 0.000005
- joint base_link_left head camera_joint: origin xyz=0.46325 0.045111 0.029551 rpy=-0.158862 0.433786 -0.408004 -> xyz=0.46325 0.045111 0.029551 rpy=-1.729658 0.433786 -1.9788
- joint base_link_rear camera_joint: origin xyz=-0.448136 -0.018115 0.012558 rpy=0.000015 0.474984 -3.141579 -> xyz=-0.448136 -0.018115 0.012558 rpy=-1.570781 0.474984 -4.712375
- joint base_link_right flank camera_joint: origin xyz=-0.135678 -0.110163 0.06561 rpy=0.000005 0.413171 -1.570794 -> xyz=-0.135678 -0.110163 0.06561 rpy=-1.570791 0.413171 -3.141591
- joint base_link_right head camera_joint: origin xyz=0.462603 -0.044896 0.027972 rpy=0.193959 0.3931 0.409605 -> xyz=0.462603 -0.044896 0.027972 rpy=-1.376837 0.3931 -1.161192
- joint front left piston motor: child solid_4 -> solid_3
- joint front right piston motor: child solid_3 -> solid_2
- joint rear left piston motor: child solid_2 -> solid_1
- joint rear right piston motor: child solid_1 -> solid_0

Commit message: update moveit for new arm
*retract arm at the beginning

File: resource/rd_spot.urdf (robot description, URDF)
Before this commit: robot /home/skpawar1305/Desktop/simulated_spot/src/webots_ros2_spot_maskor/resource/rd_spot.urdf, 77 links, 76 joints
Joints:
- joint Slider11: axis 0 0 1 -> 1 0 0
- joint spotarm_3_joint: limit lower=0 upper=2.61799 effort=500 velocity=0.5 -> lower=0 upper=3.0 effort=500 velocity=0.5

Commit message: add virtual link at the centre of the gripper

File: resource/rd_spot.urdf (robot description, URDF)
Before this commit: robot /home/skpawar1305/Desktop/simulated_spot/src/webots_ros2_spot_maskor/resource/rd_spot.urdf, 77 links, 76 joints
Links:
- added link gripper_centre; visual sphere radius=0.01
Joints:
- added joint gripper_centre_joint: type fixed, parent front, child gripper_centre, origin xyz=0 0 -0.18 rpy=0 0 0

Commit message: try blocksworld without prepublished transforms

File: resource/rd_spot.urdf (robot description, URDF)
Before this commit: robot Spot, 78 links, 77 joints
Links:
- added link gripper_camera
Joints:
- added joint spotarm_link6_gripper camera_joint: type fixed, parent spotarm_link6, child gripper_camera, origin xyz=0.19 0 0 rpy=-1.570796 0 -1.570796

Commit message: urdf converted from proto by webots has one more buggy frame, fix it manually

File: resource/rd_spot.urdf (robot description, URDF)
Before this commit: robot Spot, 78 links, 77 joints
Joints:
- joint base_link_rear depth_joint: origin xyz=-0.278136 -1.397633 0.628752 rpy=0.000015 0.474984 -3.141579 -> xyz=-0.448136 -0.018115 0.012558 rpy=0.000015 0.474984 -3.141579
