Commit message: replace landolts with hazmat signs; use perception for motion plan

File: resource/gen3.urdf (robot description, URDF)
Before this commit: robot Gen3, 24 links, 23 joints
Links:
- removed link camera_color_frame
- removed link camera_depth_frame
- added link kinova_color
- added link kinova_depth
Joints:
- joint color_module: child camera_color_frame -> kinova_color; origin xyz=0 0.05639 -0.00305 rpy=3.14159265358979 3.14159265358979 0 -> xyz=0 0.05639 -0.00305 rpy=-1.56 -1.56 0
- joint depth_module: child camera_depth_frame -> kinova_depth; origin xyz=0.0275 0.066 -0.00305 rpy=3.14159265358979 3.14159265358979 0 -> xyz=0.0275 0.066 -0.00305 rpy=-1.56 -1.56 0

File: resource/spot.urdf (robot description, URDF)
Before this commit: robot Spot, 90 links, 89 joints
Links:
- removed link camera_color_frame
- removed link camera_depth_frame
- removed link kinect range
- added link kinect_range
- added link kinova_color
- added link kinova_depth
Joints:
- joint color_module: child camera_color_frame -> kinova_color; origin xyz=0 0.05639 -0.00305 rpy=3.14159265358979 3.14159265358979 0 -> xyz=0 0.05639 -0.00305 rpy=-1.56 -1.56 0
- joint depth_module: child camera_depth_frame -> kinova_depth; origin xyz=0.0275 0.066 -0.00305 rpy=3.14159265358979 3.14159265358979 0 -> xyz=0.0275 0.066 -0.00305 rpy=-1.56 -1.56 0
- joint solid_kinect range_joint: child kinect range -> kinect_range
