Commit message: use ros2_control for manipulator and gripper

File: resource/spot.urdf (robot description, URDF)
Before this commit: robot Spot, 0 links, 0 joints
Links:
- added link SpotArm; collision cylinder length=0.035 radius=0.075; visual cylinder length=0.035 radius=0.075
- added link Velodyne_Puck; collision cylinder length=0.0727 radius=0.052; visual cylinder length=0.0727 radius=0.052
- added link accelerometer
- added link base_link; collision box size=0.030189 0.064528 0.182264; collision box size=0.030189 0.064528 0.182264
- added link cap screw
- added link cap screw(1)
- added link cap screw(10)
- added link cap screw(11)
- added link cap screw(12)
- added link cap screw(13)
- added link cap screw(14)
- added link cap screw(15)
- added link cap screw(16)
- added link cap screw(17)
- added link cap screw(18)
- added link cap screw(19)
- added link cap screw(2)
- added link cap screw(3)
- added link cap screw(4)
- added link cap screw(5)
- added link cap screw(6)
- added link cap screw(7)
- added link cap screw(8)
- added link cap screw(9)
- added link front; collision box size=0.04 0.0217 0.105; collision box size=0.04 0.0217 0.105
- added link front left forearm; collision box size=0.010189 0.05283 0.00717; collision box size=0.019245 0.071698 0.017358
- added link front left shoulder; collision box size=0.086792 0.124528 0.120755; collision box size=0.098113 0.098113 0.098113
- added link front left touch sensor
- added link front left upperarm; collision box size=0.004528 0.173585 0.015094; collision box size=0.004528 0.173585 0.015094
- added link front right forearm; collision box size=0.010189 0.05283 0.00717; collision box size=0.019245 0.071698 0.017358
- added link front right shoulder; collision box size=0.086792 0.124528 0.120755; collision box size=0.098113 0.098113 0.098113
- added link front right touch sensor
- added link front right upperarm; collision box size=0.004528 0.173585 0.015094; collision box size=0.004528 0.173585 0.015094
- added link gps
- added link gripper_centre; visual sphere radius=0.01
- added link gripper_left_finger_link; collision box size=0.0055 0.0295 0.018; collision box size=0.0076 0.05091 0.08982
- added link gripper_right_finger_link; collision box size=0.0055 0.0295 0.018; collision box size=0.0076 0.05091 0.08982
- added link gyro
- added link inertial unit
- added link kinect color
- added link kinect range
- added link left bottom led
- added link left flank camera
- added link left flank depth
- added link left head camera
- added link left head depth
- added link left middle down led
- added link left middle up led
- added link left top led
- added link rear camera
- added link rear depth
- added link rear left forearm; collision box size=0.010189 0.05283 0.00717; collision box size=0.019245 0.071698 0.017358
- added link rear left shoulder; collision box size=0.086792 0.124528 0.120755; collision box size=0.098113 0.098113 0.098113
- added link rear left touch sensor
- added link rear left upperarm; collision box size=0.004528 0.173585 0.015094; collision box size=0.004528 0.173585 0.015094
- added link rear right forearm; collision box size=0.010189 0.05283 0.00717; collision box size=0.019245 0.071698 0.017358
- added link rear right shoulder; collision box size=0.086792 0.124528 0.120755; collision box size=0.098113 0.098113 0.098113
- added link rear right touch sensor
- added link rear right upperarm; collision box size=0.004528 0.173585 0.015094; collision box size=0.004528 0.173585 0.015094
- added link right bottom led
- added link right flank camera
- added link right flank depth
- added link right head camera
- added link right head depth
- added link right middle down led
- added link right middle up led
- added link right top led
- added link solid
- added link solid_0
- added link solid_1
- added link solid_2
- added link solid_3
- added link spotarm_link1; collision box size=0.14 0.01 0.08; collision box size=0.14 0.01 0.08
- added link spotarm_link2; collision box size=0.06 0.059 0.093; collision cylinder length=0.24 radius=0.0456
- added link spotarm_link3; collision box size=0.16 0.041 0.04; collision cylinder length=0.059 radius=0.0477
- added link spotarm_link4
- added link spotarm_link5; collision box size=0.04 0.044 0.042; collision cylinder length=0.21 radius=0.0477
- added link spotarm_link6; collision cylinder length=0.065 radius=0.0477; visual cylinder length=0.065 radius=0.0477
Joints:
- added joint Slider11: type prismatic, parent spotarm_link4, child spotarm_link5, origin xyz=0.035 0 0 rpy=0 0 0, axis 1 0 0, limit lower=0 upper=0.075 effort=100 velocity=100
- added joint base_link_SpotArm_joint: type fixed, parent base_link, child SpotArm, origin xyz=0.35 0 0.1118 rpy=-0.000017 -0.000003 0.000005
- added joint base_link_Velodyne_Puck_joint: type fixed, parent base_link, child Velodyne_Puck, origin xyz=-0.063 0 0.1518 rpy=-0.000008 -0.000008 0.000001
- added joint base_link_accelerometer_joint: type fixed, parent base_link, child accelerometer, origin xyz=0 0 0 rpy=0 0 0
- added joint base_link_gps_joint: type fixed, parent base_link, child gps, origin xyz=0 0 0 rpy=0 0 0
- added joint base_link_gyro_joint: type fixed, parent base_link, child gyro, origin xyz=0 0 0 rpy=0 0 0
- added joint base_link_inertial unit_joint: type fixed, parent base_link, child inertial unit, origin xyz=0 0 0 rpy=0 0 0
- added joint base_link_left bottom led_joint: type fixed, parent base_link, child left bottom led, origin xyz=0.481728 0.081967 0.001191 rpy=1.873112 0.329178 0.767486
- added joint base_link_left flank camera_joint: type fixed, parent base_link, child left flank camera, origin xyz=-0.13568 0.110127 0.065528 rpy=-1.570799 0.403191 0.000005
- added joint base_link_left flank depth_joint: type fixed, parent base_link, child left flank depth, origin xyz=-0.13568 0.110127 0.065528 rpy=-0.000003 0.403191 1.570802
- added joint base_link_left head camera_joint: type fixed, parent base_link, child left head camera, origin xyz=0.46325 0.045111 0.029551 rpy=-1.729658 0.433786 -1.9788
- added joint base_link_left head depth_joint: type fixed, parent base_link, child left head depth, origin xyz=0.46325 0.045111 0.029551 rpy=-0.158862 0.433786 -0.408004
- added joint base_link_left middle down led_joint: type fixed, parent base_link, child left middle down led, origin xyz=0.489879 0.081966 0.018291 rpy=1.873112 0.329178 0.767486
- added joint base_link_left middle up led_joint: type fixed, parent base_link, child left middle up led, origin xyz=0.497601 0.081967 0.034491 rpy=1.873112 0.329178 0.767486
- added joint base_link_left top led_joint: type fixed, parent base_link, child left top led, origin xyz=0.505323 0.081967 0.050721 rpy=1.873112 0.329178 0.767486
- added joint base_link_rear camera_joint: type fixed, parent base_link, child rear camera, origin xyz=-0.448136 -0.018115 0.012558 rpy=-1.570781 0.474984 -4.712375
- added joint base_link_rear depth_joint: type fixed, parent base_link, child rear depth, origin xyz=-0.448136 -0.018115 0.012558 rpy=0.000015 0.474984 -3.141579
- added joint base_link_right bottom led_joint: type fixed, parent base_link, child right bottom led, origin xyz=0.481728 -0.081963 0.001193 rpy=1.279539 0.338923 -0.733718
- added joint base_link_right flank camera_joint: type fixed, parent base_link, child right flank camera, origin xyz=-0.135678 -0.110163 0.06561 rpy=-1.570791 0.413171 -3.141591
- added joint base_link_right flank depth_joint: type fixed, parent base_link, child right flank depth, origin xyz=-0.135678 -0.110163 0.06561 rpy=0.000005 0.413171 -1.570794
- added joint base_link_right head camera_joint: type fixed, parent base_link, child right head camera, origin xyz=0.462603 -0.044896 0.027972 rpy=-1.376837 0.3931 -1.161192
- added joint base_link_right head depth_joint: type fixed, parent base_link, child right head depth, origin xyz=0.462603 -0.044896 0.027972 rpy=0.193959 0.3931 0.409605
- added joint base_link_right middle down led_joint: type fixed, parent base_link, child right middle down led, origin xyz=0.489879 -0.081963 0.018293 rpy=1.279539 0.338923 -0.733718
- added joint base_link_right middle up led_joint: type fixed, parent base_link, child right middle up led, origin xyz=0.497601 -0.081963 0.034493 rpy=1.279539 0.338923 -0.733718
- added joint base_link_right top led_joint: type fixed, parent base_link, child right top led, origin xyz=0.505323 -0.081963 0.050723 rpy=1.279539 0.338923 -0.733718
- added joint base_link_solid_joint: type fixed, parent base_link, child solid, origin xyz=0.496831 0.000001 0.104801 rpy=1.2208 -0.00001 -1.570793
- added joint front left elbow motor: type revolute, parent front left upperarm, child front left forearm, origin xyz=-0.1122 -0.319729 0.182338 rpy=0 0 0, axis 1 0 0, limit lower=-0.45 upper=1.6 effort=50 velocity=10
- added joint front left forearm_front left touch sensor_joint: type fixed, parent front left forearm, child front left touch sensor, origin xyz=0.001038 -0.271321 -0.225038 rpy=-1.5708 0 1.570801
- added joint front left piston motor: type continuous, parent front left upperarm, child solid_3, origin xyz=-0.1172 -0.29077 0.2083 rpy=-0.5236 0 0, axis 1 0 0, limit effort=10 velocity=10
- added joint front left shoulder abduction motor: type revolute, parent base_link, child front left shoulder, origin xyz=0.3635 0.0528 0.012399 rpy=1.5708 -0.00001 -1.570793, axis 0 0 1, limit lower=-0.6 upper=0.5 effort=50 velocity=10
- added joint front left shoulder rotation motor: type revolute, parent front left shoulder, child front left upperarm, origin xyz=0 -0.00053 0 rpy=0 0 0, axis 1 0 0, limit lower=-1.7 upper=1.7 effort=50 velocity=10
- added joint front right elbow motor: type revolute, parent front right upperarm, child front right forearm, origin xyz=0.1122 -0.319729 0.182338 rpy=0 0 0, axis 1 0 0, limit lower=-0.45 upper=1.6 effort=50 velocity=10
- added joint front right forearm_front right touch sensor_joint: type fixed, parent front right forearm, child front right touch sensor, origin xyz=0.001038 -0.271321 -0.225038 rpy=-1.5708 0 1.570801
- added joint front right piston motor: type continuous, parent front right upperarm, child solid_2, origin xyz=0.1172 -0.29077 0.2083 rpy=-0.5236 0 0, axis 1 0 0, limit effort=10 velocity=10
- added joint front right shoulder abduction motor: type revolute, parent base_link, child front right shoulder, origin xyz=0.3635 -0.0528 0.012401 rpy=1.5708 -0.00001 -1.570793, axis 0 0 1, limit lower=-0.6 upper=0.5 effort=50 velocity=10
- added joint front right shoulder rotation motor: type revolute, parent front right shoulder, child front right upperarm, origin xyz=0 -0.00053 0 rpy=0 0 0, axis 1 0 0, limit lower=-1.7 upper=1.7 effort=50 velocity=10
- added joint front_cap screw(1)_joint: type fixed, parent front, child cap screw(1), origin xyz=0.0477 0.008 -0.043 rpy=3.141593 -1.570793 3.141593
- added joint front_cap screw(10)_joint: type fixed, parent front, child cap screw(10), origin xyz=-0.0477 -0.008 -0.043 rpy=3.141593 1.570793 3.141593
- added joint front_cap screw(11)_joint: type fixed, parent front, child cap screw(11), origin xyz=-0.0477 -0.008 -0.0108 rpy=3.141593 1.570793 3.141593
- added joint front_cap screw(12)_joint: type fixed, parent front, child cap screw(12), origin xyz=-0.0425 0.0094 -0.0945 rpy=0 0 0
- added joint front_cap screw(13)_joint: type fixed, parent front, child cap screw(13), origin xyz=0.0426 -0.0094 -0.09448 rpy=0 0 0
- added joint front_cap screw(14)_joint: type fixed, parent front, child cap screw(14), origin xyz=0 -0.033 0.0026 rpy=3.14159 0 0
- added joint front_cap screw(15)_joint: type fixed, parent front, child cap screw(15), origin xyz=0 0.033 0.0026 rpy=3.14159 0 0
- added joint front_cap screw(16)_joint: type fixed, parent front, child cap screw(16), origin xyz=-0.0433 -0.0315 0.0026 rpy=3.14159 0 0
- added joint front_cap screw(17)_joint: type fixed, parent front, child cap screw(17), origin xyz=0.0433 0.0315 0.0026 rpy=3.14159 0 0
- added joint front_cap screw(18)_joint: type fixed, parent front, child cap screw(18), origin xyz=-0.0415 0.0029 -0.0004 rpy=3.14159 0 0
- added joint front_cap screw(19)_joint: type fixed, parent front, child cap screw(19), origin xyz=0.0415 -0.0029 -0.0004 rpy=3.14159 0 0
- added joint front_cap screw(2)_joint: type fixed, parent front, child cap screw(2), origin xyz=0.0477 0.008 -0.075 rpy=3.141593 -1.570793 3.141593
- added joint front_cap screw(3)_joint: type fixed, parent front, child cap screw(3), origin xyz=0.0477 -0.008 -0.075 rpy=3.141593 -1.570793 3.141593
- added joint front_cap screw(4)_joint: type fixed, parent front, child cap screw(4), origin xyz=0.0477 -0.008 -0.043 rpy=3.141593 -1.570793 3.141593
- added joint front_cap screw(5)_joint: type fixed, parent front, child cap screw(5), origin xyz=0.0477 -0.008 -0.0108 rpy=3.141593 -1.570793 3.141593
- added joint front_cap screw(6)_joint: type fixed, parent front, child cap screw(6), origin xyz=-0.0477 0.008 -0.0108 rpy=3.141593 1.570793 3.141593
- added joint front_cap screw(7)_joint: type fixed, parent front, child cap screw(7), origin xyz=-0.0477 0.008 -0.043 rpy=3.141593 1.570793 3.141593
- added joint front_cap screw(8)_joint: type fixed, parent front, child cap screw(8), origin xyz=-0.0477 0.008 -0.075 rpy=3.141593 1.570793 3.141593
- added joint front_cap screw(9)_joint: type fixed, parent front, child cap screw(9), origin xyz=-0.0477 -0.008 -0.075 rpy=3.141593 1.570793 3.141593
- added joint front_cap screw_joint: type fixed, parent front, child cap screw, origin xyz=0.0477 0.008 -0.0108 rpy=3.141593 -1.570793 3.141593
- added joint gripper_centre_joint: type fixed, parent front, child gripper_centre, origin xyz=0 0 -0.18 rpy=0 0 0
- added joint gripper_left_finger_joint: type prismatic, parent front, child gripper_left_finger_link, origin xyz=0 0 0 rpy=0 0 3.1415, axis 1 0.000093 0, limit lower=0 upper=0.045 effort=16 velocity=0.05
- added joint gripper_right_finger_joint: type prismatic, parent front, child gripper_right_finger_link, origin xyz=0 0.0005 -0.007 rpy=0 0 0, axis 1 0 0, limit lower=0 upper=0.045 effort=16 velocity=0.05
- added joint rear left elbow motor: type revolute, parent rear left upperarm, child rear left forearm, origin xyz=-0.1122 -0.319729 0.182338 rpy=0 0 0, axis 1 0 0, limit lower=-0.45 upper=1.6 effort=50 velocity=10
- added joint rear left forearm_rear left touch sensor_joint: type fixed, parent rear left forearm, child rear left touch sensor, origin xyz=0.001038 -0.271321 -0.225038 rpy=-1.5708 0 1.570801
- added joint rear left piston motor: type continuous, parent rear left upperarm, child solid_1, origin xyz=-0.1172 -0.29077 0.2083 rpy=-0.5236 0 0, axis 1 0 0, limit effort=10 velocity=10
- added joint rear left shoulder abduction motor: type revolute, parent base_link, child rear left shoulder, origin xyz=-0.3084 0.0528 0.012299 rpy=1.5708 -0.00001 -1.570793, axis 0 0 1, limit lower=-0.6 upper=0.5 effort=50 velocity=10
- added joint rear left shoulder rotation motor: type revolute, parent rear left shoulder, child rear left upperarm, origin xyz=0 -0.00053 0 rpy=0 0 0, axis 1 0 0, limit lower=-1.7 upper=1.7 effort=50 velocity=10
- added joint rear right elbow motor: type revolute, parent rear right upperarm, child rear right forearm, origin xyz=0.1122 -0.319729 0.182338 rpy=0 0 0, axis 1 0 0, limit lower=-0.45 upper=1.6 effort=50 velocity=10
- added joint rear right forearm_rear right touch sensor_joint: type fixed, parent rear right forearm, child rear right touch sensor, origin xyz=0.001038 -0.271321 -0.225038 rpy=-1.5708 0 1.570801
- added joint rear right piston motor: type continuous, parent rear right upperarm, child solid_0, origin xyz=0.1172 -0.29077 0.2083 rpy=-0.5236 0 0, axis 1 0 0, limit effort=10 velocity=10
- added joint rear right shoulder abduction motor: type revolute, parent base_link, child rear right shoulder, origin xyz=-0.3084 -0.0528 0.012301 rpy=1.5708 -0.00001 -1.570793, axis 0 0 1, limit lower=-0.6 upper=0.5 effort=50 velocity=10
- added joint rear right shoulder rotation motor: type revolute, parent rear right shoulder, child rear right upperarm, origin xyz=0 -0.00053 0 rpy=0 0 0, axis 1 0 0, limit lower=-1.7 upper=1.7 effort=50 velocity=10
- added joint solid_kinect color_joint: type fixed, parent solid, child kinect color, origin xyz=0 0 -0.0127 rpy=-2.356193 1.570792 -0.7854
- added joint solid_kinect range_joint: type fixed, parent solid, child kinect range, origin xyz=0 0 -0.0127 rpy=-0.785397 1.570792 0.785397
- added joint spotarm_1_joint: type revolute, parent SpotArm, child spotarm_link1, origin xyz=0 0 0.04 rpy=0 0 0, axis 0 0 1, limit lower=-2.61799 upper=3.14159 effort=500 velocity=0.5
- added joint spotarm_2_joint: type revolute, parent spotarm_link1, child spotarm_link2, origin xyz=0 0.03 0.1 rpy=0 0 0, axis 0 -1 0, limit lower=-0.523599 upper=3.14159 effort=500 velocity=0.5
- added joint spotarm_3_joint: type revolute, parent spotarm_link2, child spotarm_link3, origin xyz=0.3385 -0.02 0.000137 rpy=0 0 0, axis 0 1 0, limit lower=0 upper=3.0 effort=500 velocity=0.5
- added joint spotarm_4_joint: type revolute, parent spotarm_link3, child spotarm_link4, origin xyz=0.107 -0.01 0.09734 rpy=0 0 0, axis 1 0 0, limit lower=-4.3633 upper=1.22173 effort=500 velocity=0.5
- added joint spotarm_5_joint: type revolute, parent spotarm_link5, child spotarm_link6, origin xyz=0.2413 0.01 0 rpy=0 0 0, axis 0 1 0, limit lower=-1.0472 upper=1.0472 effort=500 velocity=0.5
- added joint spotarm_6_joint: type revolute, parent spotarm_link6, child front, origin xyz=0.1 -0.0105 0 rpy=3.141593 -1.570793 3.141593, axis 0.000004 0 1, limit lower=-4.45059 upper=1.30899 effort=500 velocity=0.5

Commit message: fixup the gologpp blocksworld example

File: resource/spot.urdf (robot description, URDF)
Before this commit: robot Spot, 78 links, 77 joints
Joints:
- joint spotarm_1_joint: limit lower=-2.61799 upper=3.14159 effort=500 velocity=0.5 -> lower=-2.61799 upper=3.14159 effort=500 velocity=2.5
- joint spotarm_2_joint: limit lower=-0.523599 upper=3.14159 effort=500 velocity=0.5 -> lower=-0.523599 upper=3.14159 effort=500 velocity=2.5
- joint spotarm_3_joint: limit lower=0 upper=3.0 effort=500 velocity=0.5 -> lower=0 upper=3.0 effort=500 velocity=2.5
- joint spotarm_4_joint: limit lower=-4.3633 upper=1.22173 effort=500 velocity=0.5 -> lower=-4.3633 upper=1.22173 effort=500 velocity=2.5
- joint spotarm_5_joint: limit lower=-1.0472 upper=1.0472 effort=500 velocity=0.5 -> lower=-1.0472 upper=1.0472 effort=500 velocity=2.5
- joint spotarm_6_joint: limit lower=-4.45059 upper=1.30899 effort=500 velocity=0.5 -> lower=-4.45059 upper=1.30899 effort=500 velocity=2.5

Commit message: moveit with spot's pitch

File: resource/spot.urdf (robot description, URDF)
Before this commit: robot Spot, 78 links, 77 joints
Links:
- added link virtual_base_link
Joints:
- added joint virtual_base_link_base_link: type revolute, parent virtual_base_link, child base_link, axis 0 1 0, limit lower=-0.3 upper=0.3 effort=500 velocity=2.5
