Commit message: urdf parser throws error if links are missing in the control urdf
prepare for jazzy

File: resource/spot.urdf (robot description, URDF)
Before this commit: robot Spot, 78 links, 77 joints
Links:
- removed link SpotArm
- removed link Velodyne_Puck
- removed link accelerometer
- removed link base_link
- removed link cap screw
- removed link cap screw(1)
- removed link cap screw(10)
- removed link cap screw(11)
- removed link cap screw(12)
- removed link cap screw(13)
- removed link cap screw(14)
- removed link cap screw(15)
- removed link cap screw(16)
- removed link cap screw(17)
- removed link cap screw(18)
- removed link cap screw(19)
- removed link cap screw(2)
- removed link cap screw(3)
- removed link cap screw(4)
- removed link cap screw(5)
- removed link cap screw(6)
- removed link cap screw(7)
- removed link cap screw(8)
- removed link cap screw(9)
- removed link front
- removed link front left forearm
- removed link front left shoulder
- removed link front left touch sensor
- removed link front left upperarm
- removed link front right forearm
- removed link front right shoulder
- removed link front right touch sensor
- removed link front right upperarm
- removed link gps
- removed link gripper_centre
- removed link gripper_left_finger_link
- removed link gripper_right_finger_link
- removed link gyro
- removed link inertial unit
- removed link kinect color
- removed link kinect range
- removed link left bottom led
- removed link left flank camera
- removed link left flank depth
- removed link left head camera
- removed link left head depth
- removed link left middle down led
- removed link left middle up led
- removed link left top led
- removed link rear camera
- removed link rear depth
- removed link rear left forearm
- removed link rear left shoulder
- removed link rear left touch sensor
- removed link rear left upperarm
- removed link rear right forearm
- removed link rear right shoulder
- removed link rear right touch sensor
- removed link rear right upperarm
- removed link right bottom led
- removed link right flank camera
- removed link right flank depth
- removed link right head camera
- removed link right head depth
- removed link right middle down led
- removed link right middle up led
- removed link right top led
- removed link solid
- removed link solid_0
- removed link solid_1
- removed link solid_2
- removed link solid_3
- removed link spotarm_link1
- removed link spotarm_link2
- removed link spotarm_link3
- removed link spotarm_link4
- removed link spotarm_link5
- removed link spotarm_link6
Joints:
- removed joint Slider11
- removed joint base_link_SpotArm_joint
- removed joint base_link_Velodyne_Puck_joint
- removed joint base_link_accelerometer_joint
- removed joint base_link_gps_joint
- removed joint base_link_gyro_joint
- removed joint base_link_inertial unit_joint
- removed joint base_link_left bottom led_joint
- removed joint base_link_left flank camera_joint
- removed joint base_link_left flank depth_joint
- removed joint base_link_left head camera_joint
- removed joint base_link_left head depth_joint
- removed joint base_link_left middle down led_joint
- removed joint base_link_left middle up led_joint
- removed joint base_link_left top led_joint
- removed joint base_link_rear camera_joint
- removed joint base_link_rear depth_joint
- removed joint base_link_right bottom led_joint
- removed joint base_link_right flank camera_joint
- removed joint base_link_right flank depth_joint
- removed joint base_link_right head camera_joint
- removed joint base_link_right head depth_joint
- removed joint base_link_right middle down led_joint
- removed joint base_link_right middle up led_joint
- removed joint base_link_right top led_joint
- removed joint base_link_solid_joint
- removed joint front left elbow motor
- removed joint front left forearm_front left touch sensor_joint
- removed joint front left piston motor
- removed joint front left shoulder abduction motor
- removed joint front left shoulder rotation motor
- removed joint front right elbow motor
- removed joint front right forearm_front right touch sensor_joint
- removed joint front right piston motor
- removed joint front right shoulder abduction motor
- removed joint front right shoulder rotation motor
- removed joint front_cap screw(1)_joint
- removed joint front_cap screw(10)_joint
- removed joint front_cap screw(11)_joint
- removed joint front_cap screw(12)_joint
- removed joint front_cap screw(13)_joint
- removed joint front_cap screw(14)_joint
- removed joint front_cap screw(15)_joint
- removed joint front_cap screw(16)_joint
- removed joint front_cap screw(17)_joint
- removed joint front_cap screw(18)_joint
- removed joint front_cap screw(19)_joint
- removed joint front_cap screw(2)_joint
- removed joint front_cap screw(3)_joint
- removed joint front_cap screw(4)_joint
- removed joint front_cap screw(5)_joint
- removed joint front_cap screw(6)_joint
- removed joint front_cap screw(7)_joint
- removed joint front_cap screw(8)_joint
- removed joint front_cap screw(9)_joint
- removed joint front_cap screw_joint
- removed joint gripper_centre_joint
- removed joint gripper_left_finger_joint
- removed joint gripper_right_finger_joint
- removed joint rear left elbow motor
- removed joint rear left forearm_rear left touch sensor_joint
- removed joint rear left piston motor
- removed joint rear left shoulder abduction motor
- removed joint rear left shoulder rotation motor
- removed joint rear right elbow motor
- removed joint rear right forearm_rear right touch sensor_joint
- removed joint rear right piston motor
- removed joint rear right shoulder abduction motor
- removed joint rear right shoulder rotation motor
- removed joint solid_kinect color_joint
- removed joint solid_kinect range_joint
- removed joint spotarm_1_joint
- removed joint spotarm_2_joint
- removed joint spotarm_3_joint
- removed joint spotarm_4_joint
- removed joint spotarm_5_joint
- removed joint spotarm_6_joint

Commit message: initial commit for mesh nav added launch file mesh_nav_launch to start example world in webots modified spot_driver.py to used TwistStamped added .dae and .h5 maps

File: resource/spot.urdf (robot description, URDF)
Before this commit: robot Spot, 78 links, 77 joints
Joints:
- joint base_link_Velodyne_Puck_joint: origin xyz=-0.063 0 0.1518 rpy=-0.000008 -0.000008 0.000001 -> xyz=0.45 0 0.1518 rpy=-0.000008 -0.000008 0.000001

Commit message: add kinova in arena

File: resource/spot.urdf (robot description, URDF)
Before this commit: robot Spot, 78 links, 77 joints
Links:
- removed link SpotArm
- removed link gripper_centre
- removed link gripper_left_finger_link
- removed link gripper_right_finger_link
- removed link kinect range
- removed link spotarm_link1
- removed link spotarm_link2
- removed link spotarm_link3
- removed link spotarm_link4
- removed link spotarm_link5
- removed link spotarm_link6
- added link bicep_link, mass 1.262; collision mesh filename=package://kortex_description/arms/gen3/6dof/meshes/bicep_li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; visual mesh filename=package://kortex_description/arms/gen3/6dof/meshes/bicep_li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
- added link bracelet_link, mass 0.5; collision mesh filename=package://kortex_description/arms/gen3/6dof/meshes/bracelet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; visual mesh filename=package://kortex_description/arms/gen3/6dof/meshes/bracelet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
- added link camera_link
- added link end_effector_link, mass 0
- added link forearm_link, mass 0.93; collision mesh filename=package://kortex_description/arms/gen3/6dof/meshes/forearm_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; visual mesh filename=package://kortex_description/arms/gen3/6dof/meshes/forearm_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
- added link gen3_base_link, mass 1.697; collision mesh filename=package://kortex_description/arms/gen3/6dof/meshes/base_lin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; visual mesh filename=package://kortex_description/arms/gen3/6dof/meshes/base_lin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
- added link kinect_range
- added link kinova_color
- added link kinova_depth
- added link left_inner_finger, mass 0.0104003125914103; collision mesh filename=package://robotiq_description/meshes/collision/2f_140/robot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; visual mesh filename=package://robotiq_description/meshes/visual/2f_140/robotiq_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
- added link left_inner_finger_pad; collision box size=0.03 0.07 0.0075; visual box size=0.027 0.065 0.0075
- added link left_inner_knuckle, mass 0.0271177346495152; collision mesh filename=package://robotiq_description/meshes/collision/2f_140/robot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; visual mesh filename=package://robotiq_description/meshes/visual/2f_140/robotiq_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
- added link left_outer_finger, mass 0.022614240507152; collision mesh filename=package://robotiq_description/meshes/collision/2f_140/robot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; visual mesh filename=package://robotiq_description/meshes/visual/2f_140/robotiq_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
- added link left_outer_knuckle, mass 0.00853198276973456; collision mesh filename=package://robotiq_description/meshes/collision/2f_140/robot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; visual mesh filename=package://robotiq_description/meshes/visual/2f_140/robotiq_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
- added link right_inner_finger, mass 0.0104003125914103; collision mesh filename=package://robotiq_description/meshes/collision/2f_140/robot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; visual mesh filename=package://robotiq_description/meshes/visual/2f_140/robotiq_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
- added link right_inner_finger_pad; collision box size=0.03 0.07 0.0075; visual box size=0.027 0.065 0.0075
- added link right_inner_knuckle, mass 0.0271177346495152; collision mesh filename=package://robotiq_description/meshes/collision/2f_140/robot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; visual mesh filename=package://robotiq_description/meshes/visual/2f_140/robotiq_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
- added link right_outer_finger, mass 0.022614240507152; collision mesh filename=package://robotiq_description/meshes/collision/2f_140/robot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; visual mesh filename=package://robotiq_description/meshes/visual/2f_140/robotiq_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
- added link right_outer_knuckle, mass 0.00853198276973456; collision mesh filename=package://robotiq_description/meshes/collision/2f_140/robot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; visual mesh filename=package://robotiq_description/meshes/visual/2f_140/robotiq_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
- added link robotiq_2f_base_link, mass 0.22652; collision mesh filename=package://robotiq_description/meshes/collision/2f_140/robot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; visual mesh filename=package://robotiq_description/meshes/visual/2f_140/robotiq_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
- added link shoulder_link, mass 1.377; collision mesh filename=package://kortex_description/arms/gen3/6dof/meshes/shoulder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; visual mesh filename=package://kortex_description/arms/gen3/6dof/meshes/shoulder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
- added link spherical_wrist_1_link, mass 0.6781; collision mesh filename=package://kortex_description/arms/gen3/6dof/meshes/spherica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; visual mesh filename=package://kortex_description/arms/gen3/6dof/meshes/spherica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
- added link spherical_wrist_2_link, mass 0.678; collision mesh filename=package://kortex_description/arms/gen3/6dof/meshes/spherica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; visual mesh filename=package://kortex_description/arms/gen3/6dof/meshes/spherica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
Joints:
- removed joint Slider11
- removed joint base_link_SpotArm_joint
- removed joint gripper_centre_joint
- removed joint gripper_left_finger_joint
- removed joint gripper_right_finger_joint
- removed joint spotarm_1_joint
- removed joint spotarm_2_joint
- removed joint spotarm_3_joint
- removed joint spotarm_4_joint
- removed joint spotarm_5_joint
- removed joint spotarm_6_joint
- added joint arm_to_gripper_joint: type fixed, parent end_effector_link, child robotiq_2f_base_link, origin xyz=0 0 -0.01 rpy=0 0 1.5708
- added joint base_link_to_front: type fixed, parent base_link, child front, origin xyz=0 0 0 rpy=0 0 0
- added joint base_link_to_gen3_base_link: type fixed, parent base_link, child gen3_base_link, origin xyz=0.256 0 0.1118 rpy=0.0 0.0 0.0
- added joint camera_module: type fixed, parent end_effector_link, child camera_link, origin xyz=0 0.05639 -0.00305 rpy=3.14159265358979 3.14159265358979 0
- added joint color_module: type fixed, parent end_effector_link, child kinova_color, origin xyz=0 0.05639 -0.00305 rpy=-1.56 -1.56 0
- added joint depth_module: type fixed, parent end_effector_link, child kinova_depth, origin xyz=0.0275 0.066 -0.00305 rpy=-1.56 -1.56 0
- added joint end_effector: type fixed, parent bracelet_link, child end_effector_link, origin xyz=0 0 -0.061525 rpy=3.1416 0 -3.1416, axis 0 0 0
- added joint finger_joint: type revolute, parent robotiq_2f_base_link, child left_outer_knuckle, origin xyz=0 -0.030601 0.054905 rpy=2.2957963267948966 0 0, axis -1 0 0, limit lower=0 upper=0.8 effort=1000 velocity=2.0
- added joint joint_1: type continuous, parent gen3_base_link, child shoulder_link, origin xyz=0 0 0.15643 rpy=-3.1416 0.0 0.0, axis 0 0 1, limit effort=39 velocity=1.3963
- added joint joint_2: type revolute, parent shoulder_link, child bicep_link, origin xyz=0 0.005375 -0.12838 rpy=1.5708 0.0 0.0, axis 0 0 1, limit lower=-2.24 upper=2.24 effort=39 velocity=1.3963
- added joint joint_3: type revolute, parent bicep_link, child forearm_link, origin xyz=0 -0.41 0 rpy=3.1416 0 0, axis 0 0 1, limit lower=-3.2 upper=3.2 effort=39 velocity=1.3963
- added joint joint_4: type continuous, parent forearm_link, child spherical_wrist_1_link, origin xyz=0 0.20843 -0.006375 rpy=1.5708 0.0 0.0, axis 0 0 1, limit effort=9 velocity=1.2218
- added joint joint_5: type revolute, parent spherical_wrist_1_link, child spherical_wrist_2_link, origin xyz=0 -0.00017505 -0.10593 rpy=-1.5708 0.0 0.0, axis 0 0 1, limit lower=-2.09 upper=2.09 effort=9 velocity=1.2218
- added joint joint_6: type continuous, parent spherical_wrist_2_link, child bracelet_link, origin xyz=0 0.10593 -0.00017505 rpy=1.5708 0.0 0.0, axis 0 0 1, limit effort=9 velocity=1.2218
- added joint left_inner_finger_joint: type revolute, parent left_outer_finger, child left_inner_finger, origin xyz=0 0.0817554015893473 -0.0282203446692936 rpy=-0.725 0 0, axis 1 0 0, limit lower=-0.8757 upper=0.8757 effort=1000 velocity=2.0, mimic joint=finger_joint multiplier=1 offset=0
- added joint left_inner_finger_pad_joint: type fixed, parent left_inner_finger, child left_inner_finger_pad, origin xyz=0 0.0457554015893473 -0.0272203446692936 rpy=0 0 0, axis 0 0 1
- added joint left_inner_knuckle_joint: type revolute, parent robotiq_2f_base_link, child left_inner_knuckle, origin xyz=0 -0.0127 0.06142 rpy=2.2957963267948966 0 0.0, axis 1 0 0, limit lower=-0.8757 upper=0.8757 effort=1000 velocity=2.0, mimic joint=finger_joint multiplier=-1 offset=0
- added joint left_outer_finger_joint: type fixed, parent left_outer_knuckle, child left_outer_finger, origin xyz=0 0.01821998610742 0.0260018192872234 rpy=0 0 0, axis 1 0 0
- added joint right_inner_finger_joint: type revolute, parent right_outer_finger, child right_inner_finger, origin xyz=0 0.0817554015893473 -0.0282203446692936 rpy=-0.725 0 0, axis 1 0 0, limit lower=-0.8757 upper=0.8757 effort=1000 velocity=2.0, mimic joint=finger_joint multiplier=1 offset=0
- added joint right_inner_finger_pad_joint: type fixed, parent right_inner_finger, child right_inner_finger_pad, origin xyz=0 0.0457554015893473 -0.0272203446692936 rpy=0 0 0, axis 0 0 1
- added joint right_inner_knuckle_joint: type revolute, parent robotiq_2f_base_link, child right_inner_knuckle, origin xyz=0 0.0127 0.06142 rpy=2.2957963267948966 0 -3.141592653589793, axis 1 0 0, limit lower=-0.8757 upper=0.8757 effort=1000 velocity=2.0, mimic joint=finger_joint multiplier=-1 offset=0
- added joint right_outer_finger_joint: type fixed, parent right_outer_knuckle, child right_outer_finger, origin xyz=0 0.01821998610742 0.0260018192872234 rpy=0 0 0, axis 1 0 0
- added joint right_outer_knuckle_joint: type revolute, parent robotiq_2f_base_link, child right_outer_knuckle, origin xyz=0 0.030601 0.054905 rpy=2.2957963267948966 0 3.141592653589793, axis 1 0 0, limit lower=-0.8 upper=0.0 effort=1000 velocity=2.0, mimic joint=finger_joint multiplier=-1 offset=0
- joint base_link_solid_joint: origin xyz=0.496831 0.000001 0.104801 rpy=1.2208 -0.00001 -1.570793 -> xyz=0.496831 0.000001 0.104801 rpy=0 0 0
- joint solid_kinect color_joint: origin xyz=0 0 -0.0127 rpy=-2.356193 1.570792 -0.7854 -> xyz=0 0 -0.0127 rpy=0 0 0
- joint solid_kinect range_joint: child kinect range -> kinect_range; origin xyz=0 0 -0.0127 rpy=-0.785397 1.570792 0.785397 -> xyz=0 0 -0.0127 rpy=0 0 0

Commit message: enable color point cloud

File: resource/spot.urdf (robot description, URDF)
Before this commit: robot Spot, 90 links, 89 joints
Links:
- removed link kinect color
- removed link left flank camera
- removed link left flank depth
- removed link left head camera
- removed link left head depth
- removed link rear camera
- removed link rear depth
- removed link right flank camera
- removed link right flank depth
- removed link right head camera
- removed link right head depth
- removed link solid
- added link Kinect; collision box size=0.084 0.027 0.068; visual box size=0.084 0.027 0.068
- added link kinect_color
- added link left_flank_camera
- added link left_flank_depth
- added link left_head_camera
- added link left_head_depth
- added link rear_camera
- added link rear_depth
- added link right_flank_camera
- added link right_flank_depth
- added link right_head_camera
- added link right_head_depth
Joints:
- removed joint base_link_solid_joint
- removed joint solid_kinect color_joint
- removed joint solid_kinect range_joint
- added joint base_link_Kinect_joint: type fixed, parent base_link, child Kinect, origin xyz=0.496831 0.000001 0.104801 rpy=1.2208 -0.00001 -1.570793
- added joint kinect_color_joint: type fixed, parent Kinect, child kinect_color, origin xyz=0 0 0 rpy=3.14 0 0
- added joint kinect_range_joint: type fixed, parent Kinect, child kinect_range, origin xyz=0 0 0 rpy=3.14 0 0
- joint base_link_left flank camera_joint: child left flank camera -> left_flank_camera; origin xyz=-0.13568 0.110127 0.065528 rpy=-1.570799 0.403191 0.000005 -> xyz=-0.13568 0.110127 0.065528 rpy=-2 0 0
- joint base_link_left flank depth_joint: child left flank depth -> left_flank_depth; origin xyz=-0.13568 0.110127 0.065528 rpy=-0.000003 0.403191 1.570802 -> xyz=-0.13568 0.110127 0.065528 rpy=-2 0 0
- joint base_link_left head camera_joint: child left head camera -> left_head_camera
- joint base_link_left head depth_joint: child left head depth -> left_head_depth; origin xyz=0.46325 0.045111 0.029551 rpy=-0.158862 0.433786 -0.408004 -> xyz=-0.135678 -0.110163 0.06561 rpy=-1.729658 0.433786 -1.9788
- joint base_link_rear camera_joint: child rear camera -> rear_camera; origin xyz=-0.448136 -0.018115 0.012558 rpy=-1.570781 0.474984 -4.712375 -> xyz=-0.448136 -0.018115 0.012558 rpy=-2.03 0 1.56
- joint base_link_rear depth_joint: child rear depth -> rear_depth; origin xyz=-0.448136 -0.018115 0.012558 rpy=0.000015 0.474984 -3.141579 -> xyz=-0.448136 -0.018115 0.012558 rpy=-2.03 0 1.56
- joint base_link_right flank camera_joint: child right flank camera -> right_flank_camera; origin xyz=-0.135678 -0.110163 0.06561 rpy=-1.570791 0.413171 -3.141591 -> xyz=-0.135678 -0.110163 0.06561 rpy=-2 0 3.14
- joint base_link_right flank depth_joint: child right flank depth -> right_flank_depth; origin xyz=-0.135678 -0.110163 0.06561 rpy=0.000005 0.413171 -1.570794 -> xyz=-0.135678 -0.110163 0.06561 rpy=-2 0 3.14
- joint base_link_right head camera_joint: child right head camera -> right_head_camera
- joint base_link_right head depth_joint: child right head depth -> right_head_depth

Commit message: replace collisions with simple geometry; remove color pcl nodes

File: resource/spot.urdf (robot description, URDF)
Before this commit: robot Spot, 90 links, 89 joints
Joints:
- joint base_link_to_gen3_base_link: origin xyz=0.256 0 0.1118 rpy=0.0 0.0 0.0 -> xyz=0.3 0 0.08 rpy=0.0 0.0 0.0

Commit message: corrected left head joint

File: resource/spot.urdf (robot description, URDF)
Before this commit: robot Spot, 90 links, 89 joints
Joints:
- joint base_link_left head depth_joint: origin xyz=-0.135678 -0.110163 0.06561 rpy=-1.729658 0.433786 -1.9788 -> xyz=0.46325 0.045111 0.029551 rpy=-0.158862 0.433786 -0.408004

Commit message: fix tf rotations for spot depth cameras

File: resource/spot.urdf (robot description, URDF)
Before this commit: robot Spot, 90 links, 89 joints
Links:
- removed link left bottom led
- removed link left_flank_camera
- removed link left_flank_depth
- removed link left_head_camera
- removed link left_head_depth
- removed link rear_camera
- removed link rear_depth
- removed link right_flank_camera
- removed link right_flank_depth
- removed link right_head_camera
- removed link right_head_depth
- added link left flank camera
- added link left flank depth
- added link left head camera
- added link left head depth
- added link rear camera
- added link rear depth
- added link right flank camera
- added link right flank depth
- added link right head camera
- added link right head depth
Joints:
- removed joint base_link_left bottom led_joint
- joint base_link_left flank camera_joint: child left_flank_camera -> left flank camera; origin xyz=-0.13568 0.110127 0.065528 rpy=-2 0 0 -> xyz=-0.13568 0.110127 0.065528 rpy=-1.570799 0.403191 0.000005
- joint base_link_left flank depth_joint: child left_flank_depth -> left flank depth; origin xyz=-0.13568 0.110127 0.065528 rpy=-2 0 0 -> xyz=-0.13568 0.110127 0.065528 rpy=-0.000003 0.403191 1.570802
- joint base_link_left head camera_joint: child left_head_camera -> left head camera
- joint base_link_left head depth_joint: child left_head_depth -> left head depth
- joint base_link_rear camera_joint: child rear_camera -> rear camera; origin xyz=-0.448136 -0.018115 0.012558 rpy=-2.03 0 1.56 -> xyz=-0.448136 -0.018115 0.012558 rpy=-1.570781 0.474984 -4.712375
- joint base_link_rear depth_joint: child rear_depth -> rear depth; origin xyz=-0.448136 -0.018115 0.012558 rpy=-2.03 0 1.56 -> xyz=-0.448136 -0.018115 0.012558 rpy=0.000015 0.474984 -3.141579
- joint base_link_right flank camera_joint: child right_flank_camera -> right flank camera; origin xyz=-0.135678 -0.110163 0.06561 rpy=-2 0 3.14 -> xyz=-0.135678 -0.110163 0.06561 rpy=-1.570791 0.413171 -3.141591
- joint base_link_right flank depth_joint: child right_flank_depth -> right flank depth; origin xyz=-0.135678 -0.110163 0.06561 rpy=-2 0 3.14 -> xyz=-0.135678 -0.110163 0.06561 rpy=0.000005 0.413171 -1.570794
- joint base_link_right head camera_joint: child right_head_camera -> right head camera
- joint base_link_right head depth_joint: child right_head_depth -> right head depth
